File: hardware/custom-16-port-interface/custom-16-port-interface/dsp.kicad_sch (KiCad schematic)
At the start: 14 parts

Commit message: Added fpga firmware for ADAT->TDM, updated schematic
Parts:
- added R? (x2): 4k7, symbol Device:R
Connections:
- net +3.3V: now also R?.1, R?.1
- net TDM_DATA: now reaches U?.128 (DR1)
- net FSYNC: now reaches U?.129 (FSR1)
- net BCLK: now reaches U?.130 (CLKR1)
- net SDA: now reaches U?.89 (SDA)
- net SDA: now also R?.2
- net SCL: now reaches U?.90 (SCL)
- net SCL: now also R?.2
- no-connect marks 9 -> 15
Changed lines of the file:
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@@
   (junction (at 209.55 204.47) (diameter 0) (color 0 0 0 0)
   )
+  (junction (at 97.79 191.77) (diameter 0) (color 0 0 0 0)
+  )
   (junction (at 209.55 224.79) (diameter 0) (color 0 0 0 0)
   )
@@
   (junction (at 127 57.15) (diameter 0) (color 0 0 0 0)
   )
+  (junction (at 93.98 176.53) (diameter 0) (color 0 0 0 0)
+  )
   (junction (at 367.284 39.624) (diameter 0) (color 0 0 0 0)
   )
@@
   )
   (junction (at 204.47 120.65) (diameter 0) (color 0 0 0 0)
+  )
+  (junction (at 88.9 189.23) (diameter 0) (color 0 0 0 0)
   )
   (junction (at 367.284 136.652) (diameter 0) (color 0 0 0 0)
@@
   (no_connect (at 130.81 87.63))
   (no_connect (at 69.85 31.75))
+  (no_connect (at 205.74 166.37))
+  (no_connect (at 205.74 196.85))
+  (no_connect (at 205.74 176.53))
   (no_connect (at 130.81 92.71))
   (no_connect (at 130.81 77.47))
   (no_connect (at 130.81 69.85))
   (no_connect (at 201.93 113.03))
+  (no_connect (at 205.74 191.77))
   (no_connect (at 130.81 85.09))
   (no_connect (at 130.81 72.39))
+  (no_connect (at 205.74 199.39))
+  (no_connect (at 205.74 168.91))
   (no_connect (at 130.81 80.01))
   (wire (pts (xy 127 120.65) (xy 127 128.27))
@@
     (stroke (width 0) (type default) (color 0 0 0 0))
   )
+  (wire (pts (xy 86.36 191.77) (xy 97.79 191.77))
+    (stroke (width 0) (type default) (color 0 0 0 0))
+  )
   (wire (pts (xy 348.996 80.264) (xy 354.584 80.264))
     (stroke (width 0) (type default) (color 0 0 0 0))
@@
     (stroke (width 0) (type default) (color 0 0 0 0))
   )
+  (wire (pts (xy 88.9 185.42) (xy 88.9 189.23))
+    (stroke (width 0) (type default) (color 0 0 0 0))
+  )
   (wire (pts (xy 359.41 38.1) (xy 359.41 39.624))
     (stroke (width 0) (type default) (color 0 0 0 0))
@@
     (stroke (width 0) (type default) (color 0 0 0 0))
   )
+  (wire (pts (xy 88.9 177.8) (xy 88.9 176.53))
+    (stroke (width 0) (type default) (color 0 0 0 0))
+  )
   (wire (pts (xy 116.84 179.07) (xy 124.46 179.07))
     (stroke (width 0) (type default) (color 0 0 0 0))
@@
     (stroke (width 0) (type default) (color 0 0 0 0))
   )
+  (wire (pts (xy 93.98 176.53) (xy 93.98 173.99))
+    (stroke (width 0) (type default) (color 0 0 0 0))
+  )
   (wire (pts (xy 120.65 237.49) (xy 120.65 224.79))
     (stroke (width 0) (type default) (color 0 0 0 0))
@@
     (stroke (width 0) (type default) (color 0 0 0 0))
   )
+  (wire (pts (xy 97.79 177.8) (xy 97.79 176.53))
+    (stroke (width 0) (type default) (color 0 0 0 0))
+  )
   (wire (pts (xy 348.488 115.824) (xy 354.584 115.824))
     (stroke (width 0) (type default) (color 0 0 0 0))
@@
     (stroke (width 0) (type default) (color 0 0 0 0))
   )
+  (wire (pts (xy 205.74 189.23) (xy 213.36 189.23))
+    (stroke (width 0) (type default) (color 0 0 0 0))
+  )
   (wire (pts (xy 348.996 85.344) (xy 354.584 85.344))
     (stroke (width 0) (type default) (color 0 0 0 0))
@@
     (stroke (width 0) (type default) (color 0 0 0 0))
   )
+  (wire (pts (xy 88.9 189.23) (xy 124.46 189.23))
+    (stroke (width 0) (type default) (color 0 0 0 0))
+  )
   (wire (pts (xy 364.744 23.368) (xy 364.744 27.94))
     (stroke (width 0) (type default) (color 0 0 0 0))
@@
     (stroke (width 0) (type default) (color 0 0 0 0))
   )
+  (wire (pts (xy 97.79 185.42) (xy 97.79 191.77))
+    (stroke (width 0) (type default) (color 0 0 0 0))
+  )
   (wire (pts (xy 204.47 100.33) (xy 204.47 120.65))
     (stroke (width 0) (type default) (color 0 0 0 0))
@@
     (stroke (width 0) (type default) (color 0 0 0 0))
   )
+  (wire (pts (xy 97.79 191.77) (xy 124.46 191.77))
+    (stroke (width 0) (type default) (color 0 0 0 0))
+  )
   (wire (pts (xy 367.284 136.652) (xy 367.284 138.176))
     (stroke (width 0) (type default) (color 0 0 0 0))
@@
     (stroke (width 0) (type default) (color 0 0 0 0))
   )
+  (wire (pts (xy 97.79 176.53) (xy 93.98 176.53))
+    (stroke (width 0) (type default) (color 0 0 0 0))
+  )
   (wire (pts (xy 123.444 95.25) (xy 130.81 95.25))
     (stroke (width 0) (type default) (color 0 0 0 0))
@@
     (stroke (width 0) (type default) (color 0 0 0 0))
   )
+  (wire (pts (xy 88.9 176.53) (xy 93.98 176.53))
+    (stroke (width 0) (type default) (color 0 0 0 0))
+  )
+  (wire (pts (xy 86.36 189.23) (xy 88.9 189.23))
+    (stroke (width 0) (type default) (color 0 0 0 0))
+  )
+  (wire (pts (xy 205.74 186.69) (xy 213.36 186.69))
+    (stroke (width 0) (type default) (color 0 0 0 0))
+  )
   (wire (pts (xy 201.93 87.63) (xy 209.296 87.63))
     (stroke (width 0) (type default) (color 0 0 0 0))
@@
     (stroke (width 0) (type default) (color 0 0 0 0))
   )
+  (wire (pts (xy 205.74 184.15) (xy 213.36 184.15))
+    (stroke (width 0) (type default) (color 0 0 0 0))
+  )
   (wire (pts (xy 201.93 62.23) (xy 204.47 62.23))
     (stroke (width 0) (type default) (color 0 0 0 0))
@@
     )
   )
+  (global_label "BCLK" (shape output) (at 213.36 184.15 0) (fields_autoplaced)
+    (effects (font (size 1.27 1.27)) (justify left))
+    (property "Intersheet References" "${INTERSHEET_REFS}" (id 0) (at 220.6112 184.0706 0)
+      (effects (font (size 1.27 1.27)) (justify left))
+    )
+  )
   (global_label "DQ13" (shape bidirectional) (at 387.604 92.964 0) (fields_autoplaced)
     (effects (font (size 1.27 1.27)) (justify left))
@@
     )
   )
+  (global_label "SCL" (shape bidirectional) (at 86.36 191.77 180) (fields_autoplaced)
+    (effects (font (size 1.27 1.27)) (justify right))
+    (property "Intersheet References" "${INTERSHEET_REFS}" (id 0) (at 80.4393 191.6906 0)
+      (effects (font (size 1.27 1.27)) (justify right))
+    )
+  )
   (global_label "~{SDCAS}" (shape output) (at 123.444 100.33 180) (fields_autoplaced)
     (effects (font (size 1.27 1.27)) (justify right))
@@
     )
   )
+  (global_label "TDM_DATA" (shape input) (at 213.36 189.23 0) (fields_autoplaced)
+    (effects (font (size 1.27 1.27)) (justify left))
+    (property "Intersheet References" "${INTERSHEET_REFS}" (id 0) (at 224.8445 189.1506 0)
+      (effects (font (size 1.27 1.27)) (justify left))
+    )
+  )
   (global_label "SDA10" (shape input) (at 348.996 92.964 180) (fields_autoplaced)
     (effects (font (size 1.27 1.27)) (justify right))
@@
     )
   )
+  (global_label "FSYNC" (shape output) (at 213.36 186.69 0) (fields_autoplaced)
+    (effects (font (size 1.27 1.27)) (justify left))
+    (property "Intersheet References" "${INTERSHEET_REFS}" (id 0) (at 221.7602 186.6106 0)
+      (effects (font (size 1.27 1.27)) (justify left))
+    )
+  )
   (global_label "~{SDCAS}" (shape input) (at 348.488 118.364 180) (fields_autoplaced)
     (effects (font (size 1.27 1.27)) (justify right))
@@
     (property "Intersheet References" "${INTERSHEET_REFS}" (id 0) (at 215.5191 57.2294 0)
       (effects (font (size 1.27 1.27)) (justify left))
+    )
+  )
+  (global_label "SDA" (shape bidirectional) (at 86.36 189.23 180) (fields_autoplaced)
+    (effects (font (size 1.27 1.27)) (justify right))
+    (property "Intersheet References" "${INTERSHEET_REFS}" (id 0) (at 80.3788 189.1506 0)
+      (effects (font (size 1.27 1.27)) (justify right))
     )
   )
@@
     )
     (property "Datasheet" "~" (id 3) (at 359.41 34.29 0)
+      (effects (font (size 1.27 1.27)) hide)
+    )
+    (pin "1")
+    (pin "2")
+  )
+  (symbol (lib_id "Device:R") (at 88.9 181.61 0) (unit 1)
+    (in_bom yes) (on_board yes) (fields_autoplaced)
+    (property "Reference" "R?" (id 0) (at 91.44 180.3399 0)
+      (effects (font (size 1.27 1.27)) (justify left))
+    )
+    (property "Value" "4k7" (id 1) (at 91.44 182.8799 0)
+      (effects (font (size 1.27 1.27)) (justify left))
+    )
+    (property "Footprint" "" (id 2) (at 87.122 181.61 90)
+      (effects (font (size 1.27 1.27)) hide)
+    )
+    (property "Datasheet" "~" (id 3) (at 88.9 181.61 0)
       (effects (font (size 1.27 1.27)) hide)
     )
@@
     (pin "99")
   )
+  (symbol (lib_id "power:+3.3V") (at 93.98 173.99 0) (unit 1)
+    (in_bom yes) (on_board yes) (fields_autoplaced)
+    (property "Reference" "#PWR?" (id 0) (at 93.98 177.8 0)
+      (effects (font (size 1.27 1.27)) hide)
+    )
+    (property "Value" "+3.3V" (id 1) (at 93.98 168.91 0))
+    (property "Footprint" "" (id 2) (at 93.98 173.99 0)
+      (effects (font (size 1.27 1.27)) hide)
+    )
+    (property "Datasheet" "" (id 3) (at 93.98 173.99 0)
+      (effects (font (size 1.27 1.27)) hide)
+    )
+    (pin "1")
+  )
   (symbol (lib_id "Device:R") (at 118.11 34.29 90) (unit 1)
     (in_bom yes) (on_board yes)
@@
     (pin "1")
   )
+  (symbol (lib_id "Device:R") (at 97.79 181.61 0) (unit 1)
+    (in_bom yes) (on_board yes) (fields_autoplaced)
+    (property "Reference" "R?" (id 0) (at 100.33 180.3399 0)
+      (effects (font (size 1.27 1.27)) (justify left))
+    )
+    (property "Value" "4k7" (id 1) (at 100.33 182.8799 0)
+      (effects (font (size 1.27 1.27)) (justify left))
+    )
+    (property "Footprint" "" (id 2) (at 96.012 181.61 90)
+      (effects (font (size 1.27 1.27)) hide)
+    )
+    (property "Datasheet" "~" (id 3) (at 97.79 181.61 0)
+      (effects (font (size 1.27 1.27)) hide)
+    )
+    (pin "1")
+    (pin "2")
+  )
   (symbol (lib_id "power:GND") (at 72.39 50.8 0) (unit 1)
